File: PCBRulerSmaller.kicad_pcb (KiCad board)
At the start: 2 copper layers, 65 x 25 mm, 25 parts

Commit message: add PCBRulerSmaller gerbers
Parts:
- moved TSSOP 13.8 mm to (117.8, 103.0)
- moved SOIC8 12.0 mm to (117.6, 115.5)
- moved SOT23 9.62 mm to (101.2, 102.8)
- moved SOT23-5 9.50 mm to (99.8, 108.2)
- moved QFN28 7.75 mm to (99.8, 113.8)
- moved 0402 2.02 mm to (95.8, 117.0)
- moved REF** 1.50 mm to (142.5, 117.3)
- moved REF** 1.50 mm to (92.5, 117.5)
- moved 0603 1.03 mm to (95.0, 113.2)
- moved BGA16 0.56 mm to (105.3, 116.5)
- moved SOT89 0.50 mm to (116.4, 108.8)
- moved SOD323 0.25 mm to (105.5, 111.0)
Other:
- board size 65 x 25 mm -> 65 x 23.5 mm
- board text added: "r= 0.5mm"
- board text removed: "r=0.5mm"
